Commit message: Update caster_diffbot.xacro

File: Programas_requeridos/urdf/caster_diffbot.xacro (robot description, xacro)
@@ -1,5 +1,5 @@
 <?xml version="1.0"?>
 <robot name="caster_diffbot" xmlns:xacro="http://ros.org/wiki/xacro">
-  <xacro:property name="package_name" value="gazebo_world_launch"/>
+  <xacro:property name="package_name" value="basic_diffbot"/>
   <xacro:property name="PI" value="3.14159265"/>
   <xacro:property name="wheelSeparation" value="0.13"/>
